File: hardware/analyzer/mula.kicad_pcb (KiCad board)
At the start: 4 copper layers, 22 x 42 mm, 46 parts, among them J101 USB_C_Receptacle_USB2.0, J102 M.2, SW101 BOOT, SW102 RESET, U101 W25Q128JVS, U102 RP2040, U103 SRV05-4, U104 XC6206, U105 SN74LVC4245, U106 SN74LVC4245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

Commit message: move things around
Parts:
- added FID101: Fiducial, Fiducial:Fiducial_0.5mm_Mask1mm, F.Cu at (129.9, 72.9)
- added FID102: Fiducial, Fiducial:Fiducial_0.5mm_Mask1mm, F.Cu at (129.9, 109.0)
- added FID103: Fiducial, Fiducial:Fiducial_0.5mm_Mask1mm, F.Cu at (150.1, 109.1)
- moved L101 5.90 mm to (133.6, 105.1)
- moved L102 5.82 mm to (146.6, 105.1)
- moved kibuzzard-64C5EFF0 1.75 mm to (140.2, 107.7)
Routing:
- net /IO0: track 18.2 -> 11.4 mm
- net /IO1: track 17.1 -> 10.5 mm
- net /IO15: track 18.0 -> 11.4 mm
- net /IO2: track 16.0 -> 9.51 mm
- net /IO14: track 16.8 -> 10.4 mm
- net /IO3: track 14.8 -> 8.55 mm
- net /IO13: track 15.7 -> 9.44 mm
- net /IO12: track 14.6 -> 8.48 mm
- net /IO4: track 13.5 -> 7.45 mm
- net GND: track 76.6 -> 82.4 mm, vias 34 -> 32
- net /IO11: track 13.2 -> 7.39 mm
- net /xIO7: track 3.51 -> 9.15 mm
- net /xIO1: track 3.27 -> 8.90 mm
- net /xIO2: track 3.31 -> 8.94 mm
- net /xIO5: track 3.43 -> 9.07 mm
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