File: hardware/analyzer/mula.kicad_sch (KiCad schematic)
At the start: 43 parts, among them J101 USB_C_Receptacle_USB2.0, J102 M.2, SW101 BOOT, SW102 RESET, U101 W25Q128JVS, U102 RP2040, U103 SRV05-4, U104 XC6206, U105 SN74LVC4245, U106 SN74LVC4245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

Commit message: move things around
Parts:
- added FID101, FID102, FID103: Fiducial, Fiducial:Fiducial_0.5mm_Mask1mm, symbol Mechanical:Fiducial
- J101: LCSC Part (none) -> C165948
- J102: now left out of the parts list
- RN101, RN102, RN103, RN104: LCSC Part (none) -> C425271
- SW101, SW102: LCSC Part (none) -> C318884
- U101: LCSC Part (none) -> C97521
- U102: LCSC Part (none) -> C2040
- U103: LCSC Part (none) -> C85364
- U104: LCSC Part (none) -> C5446
- U105, U106: LCSC Part (none) -> C7859
- Y101: LCSC Part (none) -> C9002
Changed lines of the file:
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@@
+    )
+  )
+  (symbol (lib_id "Mechanical:Fiducial") (at 269.24 219.71 0) (unit 1)
+    (in_bom no) (on_board yes) (dnp no) (fields_autoplaced)
+    (property "Reference" "FID102" (at 271.78 218.44 0)
+      (effects (font (size 1.27 1.27)) (justify left))
+    )
+    (property "Value" "Fiducial" (at 271.78 220.98 0)
+      (effects (font (size 1.27 1.27)) (justify left))
+    )
+    (property "Footprint" "Fiducial:Fiducial_0.5mm_Mask1mm" (at 269.24 219.71 0)
+      (effects (font (size 1.27 1.27)) hide)
+    )
+    (property "Datasheet" "~" (at 269.24 219.71 0)
+      (effects (font (size 1.27 1.27)) hide)
+    )
+    (instances
+      (project "mula"
+        (path "/117fe963-ddb8-44f3-995a-8e9baa48b9ed"
+          (reference "FID102") (unit 1)
+        )
+      )
     )
   )
@@
     )
     (property "Datasheet" "https://datasheets.raspberrypi.com/rp2040/rp2040-datasheet.pdf" (at 129.54 109.22 0)
+      (effects (font (size 1.27 1.27)) hide)
+    )
+    (property "LCSC Part" "C2040" (at 129.54 109.22 0)
       (effects (font (size 1.27 1.27)) hide)
     )
@@
       (effects (font (size 1.27 1.27)) hide)
     )
+    (property "LCSC Part" "C7859" (at 215.9 77.47 0)
+      (effects (font (size 1.27 1.27)) hide)
+    )
     (pin "10")
     (pin "11")
@@
       (effects (font (size 1.27 1.27)) hide)
     )
+    (property "LCSC Part" "C5446" (at 204.47 213.36 0)
+      (effects (font (size 1.27 1.27)) hide)
+    )
     (pin "1")
     (pin "2")
@@
     )
     (property "Datasheet" "http://www.winbond.com/resource-files/w25q128jv_dtr%20revc%2003272018%20plus.pdf" (at 44.45 96.52 0)
+      (effects (font (size 1.27 1.27)) hide)
+    )
+    (property "LCSC Part" "C97521" (at 44.45 96.52 0)
       (effects (font (size 1.27 1.27)) hide)
     )
@@
     )
     (property "Datasheet" "~" (at 255.27 62.23 0)
+      (effects (font (size 1.27 1.27)) hide)
+    )
+    (property "LCSC Part" "C425271" (at 255.27 62.23 0)
       (effects (font (size 1.27 1.27)) hide)
     )
@@
   )
   (symbol (lib_id "Connector_Generic:Conn_02x16_Top_Bottom") (at 342.9 106.68 180) (unit 1)
-    (in_bom yes) (on_board yes) (dnp no)
+    (in_bom no) (on_board yes) (dnp no)
     (property "Reference" "J102" (at 341.63 76.2 0)
       (effects (font (size 1.27 1.27)))
@@
       (effects (font (size 1.27 1.27)) hide)
     )
+    (property "LCSC Part" "C425271" (at 270.51 62.23 0)
+      (effects (font (size 1.27 1.27)) hide)
+    )
     (pin "1")
     (pin "2")
@@
       (effects (font (size 1.27 1.27)) hide)
     )
+    (property "LCSC Part" "C318884" (at 78.74 68.58 0)
+      (effects (font (size 1.27 1.27)) hide)
+    )
     (pin "1")
     (pin "2")
@@
     )
     (property "Datasheet" "https://datasheet.lcsc.com/lcsc/1809192324_Texas-Instruments-SN74LVC4245APWR_C7859.pdf" (at 215.9 162.56 0)
+      (effects (font (size 1.27 1.27)) hide)
+    )
+    (property "LCSC Part" "C7859" (at 215.9 133.35 0)
       (effects (font (size 1.27 1.27)) hide)
     )
@@
     )
   )
+  (symbol (lib_id "Mechanical:Fiducial") (at 269.24 226.06 0) (unit 1)
+    (in_bom no) (on_board yes) (dnp no) (fields_autoplaced)
+    (property "Reference" "FID103" (at 271.78 224.79 0)
+      (effects (font (size 1.27 1.27)) (justify left))
+    )
+    (property "Value" "Fiducial" (at 271.78 227.33 0)
+      (effects (font (size 1.27 1.27)) (justify left))
+    )
+    (property "Footprint" "Fiducial:Fiducial_0.5mm_Mask1mm" (at 269.24 226.06 0)
+      (effects (font (size 1.27 1.27)) hide)
+    )
+    (property "Datasheet" "~" (at 269.24 226.06 0)
+      (effects (font (size 1.27 1.27)) hide)
+    )
+    (instances
+      (project "mula"
+        (path "/117fe963-ddb8-44f3-995a-8e9baa48b9ed"
+          (reference "FID103") (unit 1)
+        )
+      )
+    )
+  )
   (symbol (lib_id "Device:R_Small_US") (at 96.52 78.74 90) (unit 1)
     (in_bom yes) (on_board yes) (dnp no)
@@
     )
     (property "Datasheet" "https://www.usb.org/sites/default/files/documents/usb_type-c.zip" (at 64.77 214.63 0)
+      (effects (font (size 1.27 1.27)) hide)
+    )
+    (property "LCSC Part" "C165948" (at 60.96 214.63 0)
       (effects (font (size 1.27 1.27)) hide)
     )
@@
       (effects (font (size 1.27 1.27)) hide)
     )
+    (property "LCSC Part" "C9002" (at 91.44 121.92 90)
+      (effects (font (size 1.27 1.27)) hide)
+    )
     (pin "1")
     (pin "2")
@@
       (effects (font (size 1.27 1.27)) hide)
     )
+    (property "LCSC Part" "C318884" (at 63.5 68.58 0)
+      (effects (font (size 1.27 1.27)) hide)
+    )
     (pin "1")
     (pin "2")
@@
     )
     (property "Datasheet" "http://www.onsemi.com/pub/Collateral/SRV05-4-D.PDF" (at 129.54 215.9 0)
+      (effects (font (size 1.27 1.27)) hide)
+    )
+    (property "LCSC Part" "C85364" (at 129.54 215.9 0)
       (effects (font (size 1.27 1.27)) hide)
     )
@@
     )
   )
+  (symbol (lib_id "Mechanical:Fiducial") (at 269.24 213.36 0) (unit 1)
+    (in_bom no) (on_board yes) (dnp no) (fields_autoplaced)
+    (property "Reference" "FID101" (at 271.78 212.09 0)
+      (effects (font (size 1.27 1.27)) (justify left))
+    )
+    (property "Value" "Fiducial" (at 271.78 214.63 0)
+      (effects (font (size 1.27 1.27)) (justify left))
+    )
+    (property "Footprint" "Fiducial:Fiducial_0.5mm_Mask1mm" (at 269.24 213.36 0)
+      (effects (font (size 1.27 1.27)) hide)
+    )
+    (property "Datasheet" "~" (at 269.24 213.36 0)
+      (effects (font (size 1.27 1.27)) hide)
+    )
+    (instances
+      (project "mula"
+        (path "/117fe963-ddb8-44f3-995a-8e9baa48b9ed"
+          (reference "FID101") (unit 1)
+        )
+      )
+    )
+  )
   (symbol (lib_id "Device:R_Small_US") (at 101.6 62.23 0) (mirror y) (unit 1)
     (in_bom yes) (on_board yes) (dnp no)
@@
     )
     (property "Datasheet" "~" (at 269.24 118.11 0)
+      (effects (font (size 1.27 1.27)) hide)
+    )
+    (property "LCSC Part" "C425271" (at 269.24 118.11 0)
       (effects (font (size 1.27 1.27)) hide)
     )
@@
       (effects (font (size 1.27 1.27)) hide)
     )
+    (property "LCSC Part" "C425271" (at 254 118.11 0)
+      (effects (font (size 1.27 1.27)) hide)
+    )
